Commit message: Finished template for rock_commander

File: rock_commander_robot/rock_commander_robot_description/urdf/rock_commander_base.urdf (robot description, URDF)
Before this commit: robot two_wheeled_robot, 5 links, 4 joints
Links:
- added link camera_depth_frame
- added link camera_link, mass 0.035; collision box size=0.015 0.130 0.022; visual box size=0.015 0.130 0.022
- link base_link: geometry collision box size=${base_length} ${base_width} ${base_height}; visual box size=${base_length} ${base_width} ${base_height}
- link lidar_link: geometry collision cylinder length=0.055 radius=0.0508; visual cylinder length=0.055 radius=0.0508
Joints:
- added joint camera_depth_joint: type fixed, parent camera_link, child camera_depth_frame, origin xyz=0 0 0 rpy=${-pi/2} 0 ${-pi/2}
- added joint camera_joint: type fixed, parent base_link, child camera_link, origin xyz=0.215 0 0.05 rpy=0 0 0
- joint lidar_joint: origin xyz=0.215 0.0 0.30 rpy=0 0 0 -> xyz=0 0 0.12 rpy=0 0 0
